File: ST506Pico.kicad_sch (KiCad schematic)
At the start: 9 parts, among them J1 Micro_SD_Card, J4 HD_SEL0, P1 E_CON34, P2 CON20, U1 SN74LVC245APW, U2 74ACT05

Commit message: Schematic seems to be complete. Error in MicroSD card suspected
Parts:
- added C2, C3, C4: 100n, symbol Device:C
- added J2, J6: IDC_CONN20, symbol Connector_Generic:Conn_02x10_Odd_Even
- added J3, J5: IDC_CONN34, symbol Connector_Generic:Conn_02x17_Odd_Even
- added J7: SEL, symbol Connector_Generic:Conn_02x04_Counter_Clockwise
- added R1: 100, symbol Device:R
- added R2, R3, R4: 4k7, symbol Device:R
- added RN2: 150, Resistor_THT:R_Array_SIP10, symbol Device:R_Network09
- added U3: ADM1491EBR, Package_SO:SOIC-14_3.9x8.7mm_P1.27mm, symbol Interface_UART:SN65HVD33DR
- added U4: SN74LVC245APW, Package_SO:TSSOP-20_4.4x6.5mm_P0.65mm, symbol Logic_LevelTranslator:SN74LVC245APW
- added U5, U6: 74LS05, symbol 74xx:74ACT05
Connections:
- net ~{DIR_IN} is gone; now on net DIR_IN: U1.8 (A7)
- net ~{HEAD0} is gone; now on net HEAD0: U1.5 (A4)
- net ~{HEAD1} is gone; now on net HEAD1: U1.6 (A5)
- net ~{HEAD2} is gone; now on net HEAD2: U1.3 (A2)
- net ~{HEAD3} is gone; now on net HEAD3: U1.2 (A1)
- net ~{SEL} is gone; now on net SEL1: U1.9 (A8)
- net ~{STEP} is gone; now on net STEP: U1.7 (A6)
- net ~{WRITE} is gone; now on net WRITE: U1.4 (A3)
- net +3V3: now also J1.4 (VDD), C2.1, C3.1, C4.1, R2.1, R3.1, R4.1, U3.13 (VCC), U3.14 (VCC), U4.1 (DIR), U4.20 (VCC)
- net +5V: now also RN2.1 (common)
- net E_READ+: now also J2.17 (Pin_17), U3.9 (Y)
- net E_READ-: now also J2.18 (Pin_18), U3.10 (Z)
- net E_WRITE+: now also J2.13 (Pin_13), R1.1, U3.12 (A)
- net E_WRITE-: now also J2.14 (Pin_14), R1.2, U3.11 (B)
- net GNDD: now also C2.2, C3.2, C4.2, J2.11 (Pin_11), J2.12 (Pin_12), J2.15 (Pin_15), J2.16 (Pin_16), J2.19 (Pin_19), J2.2 (Pin_2), J2.20 (Pin_20), J2.4 (Pin_4), J2.6 (Pin_6), J2.8 (Pin_8), J3.1 (Pin_1), J3.11 (Pin_11), J3.13 (Pin_13), J3.15 (Pin_15), J3.17 (Pin_17), J3.19 (Pin_19), J3.21 (Pin_21), J3.23 (Pin_23), J3.25 (Pin_25), J3.27 (Pin_27), J3.29 (Pin_29), J3.3 (Pin_3), J3.31 (Pin_31), J3.33 (Pin_33), J3.5 (Pin_5), J3.7 (Pin_7), J3.8 (Pin_8), J3.9 (Pin_9), J5.1 (Pin_1), J5.11 (Pin_11), J5.13 (Pin_13), J5.15 (Pin_15), J5.17 (Pin_17), J5.19 (Pin_19), J5.21 (Pin_21), J5.23 (Pin_23), J5.25 (Pin_25), J5.27 (Pin_27), J5.29 (Pin_29), J5.3 (Pin_3), J5.31 (Pin_31), J5.33 (Pin_33), J5.5 (Pin_5), J5.7 (Pin_7), J5.9 (Pin_9), J6.11 (Pin_11), J6.12 (Pin_12), J6.15 (Pin_15), J6.16 (Pin_16), J6.19 (Pin_19), J6.2 (Pin_2), J6.20 (Pin_20), J6.4 (Pin_4), J6.6 (Pin_6), J6.8 (Pin_8), U3.6 (GND), U3.7 (GND), U4.10 (GND)
- net INDEX: now also A1.22 (GPIO17), U4.15 (B4)
- net READY: now also A1.31 (GPIO26_ADC0), U4.14 (B5)
- net SEEKDONE: now also A1.19 (GPIO14), U4.18 (B1)
- net TRACK00: now also A1.20 (GPIO15), U4.17 (B2)
- net WRFAULT: now also A1.21 (GPIO16), U4.16 (B3)
- net ~{E_DIR_IN}: now also J3.34 (Pin_34)
- net ~{E_DRV_SEL}: now also J2.1 (Pin_1)
- net ~{E_HEAD0}: now also J3.14 (Pin_14)
- net ~{E_HEAD1}: now also J3.18 (Pin_18)
- net ~{E_HEAD2}: now also J3.4 (Pin_4)
- net ~{E_HEAD3}: now also J3.2 (Pin_2)
- net ~{E_INDEX}: now also J3.20 (Pin_20)
- net ~{E_READY}: now also J3.22 (Pin_22)
- net ~{E_SEL1}: now also J3.26 (Pin_26)
- net ~{E_SEL2}: now also J3.28 (Pin_28)
- net ~{E_SEL3}: now also J3.30 (Pin_30)
- net ~{E_SEL4}: now also J3.32 (Pin_32)
- net ~{E_STEP}: now also J3.24 (Pin_24)
- net ~{E_TRACK00}: now also J3.10 (Pin_10)
- net ~{E_WRFAULT}: now also J3.12 (Pin_12)
- net ~{E_WRITE}: now also J3.6 (Pin_6)
- net DRV_SEL: now reaches U2.13
- net DRV_SEL: now also A1.6 (GPIO4)
- net HEAD2: now reaches A1.10 (GPIO7)
- net HEAD2: now also U5.3
- net HEAD1: now reaches A1.11 (GPIO8)
- net HEAD1: now also U5.13
- net HEAD0: now reaches A1.12 (GPIO9)
- net HEAD0: now also U5.9
- net WRITE: now reaches A1.14 (GPIO10)
- net WRITE: now also U5.5
- net STEP: now reaches A1.15 (GPIO11)
- net STEP: now also U6.1
- net DIR_IN: now reaches A1.16 (GPIO12)
- net DIR_IN: now also U6.13
- net SEL1: now reaches A1.17 (GPIO13)
- net SEL1: now also U6.3
- net ~{MFM_READ_EN}: now reaches A1.32 (GPIO27_ADC1)
- net ~{MFM_READ_EN}: now also R4.2, U4.19 (~{OE})
- net SELECTED: now reaches A1.34 (GPIO28_ADC2)
- net SELECTED: now also U4.13 (B6)
- net ~{MFM0_IN}: now reaches A1.4 (GPIO2)
- net ~{MFM0_IN}: now also R2.2, U3.3 (~{RE}), U3.4 (DE)
- net MFM_DATA: now reaches A1.5 (GPIO3)
- net MFM_DATA: now also U3.2 (RO), U3.5 (DI)
- net ~{EMU_EN}: now reaches A1.7 (GPIO5)
- net ~{EMU_EN}: now also U1.19 (~{OE}), R3.2
- net HEAD3: now reaches A1.9 (GPIO6)
- net HEAD3: now also U5.1
- new net: RN2.8 (R7), U4.8 (A7)
- new net: RN2.9 (R8), U4.9 (A8)
- new net: J7.1 (Pin_1), J7.2 (Pin_2), J7.3 (Pin_3), J7.4 (Pin_4), U6.4
- new net C_READ+: J6.17 (Pin_17)
- new net C_READ-: J6.18 (Pin_18)
- new net C_WRITE+: J6.13 (Pin_13)
- new net C_WRITE-: J6.14 (Pin_14)
- new net ~{C_DIR_IN}: J5.34 (Pin_34), U6.12
- new net ~{C_DRV_SEL}: J6.1 (Pin_1), RN2.7 (R6), U4.7 (A6)
- new net ~{C_HEAD0}: J5.14 (Pin_14), U5.8
- new net ~{C_HEAD1}: J5.18 (Pin_18), U5.12
- new net ~{C_HEAD2}: J5.4 (Pin_4), U5.4
- new net ~{C_HEAD3}: J5.2 (Pin_2), U5.2
- new net ~{C_INDEX}: J5.20 (Pin_20), RN2.5 (R4), U4.5 (A4)
- new net ~{C_READY}: J5.22 (Pin_22), RN2.6 (R5), U4.6 (A5)
- new net ~{C_RECOVERY}: J5.16 (Pin_16), U5.10
- new net ~{C_SEEKDONE}: J5.8 (Pin_8), RN2.2 (R1), U4.2 (A1)
- new net ~{C_SEL1}: J5.26 (Pin_26), J7.8 (Pin_8)
- new net ~{C_SEL2}: J5.28 (Pin_28), J7.7 (Pin_7)
- new net ~{C_SEL3}: J5.30 (Pin_30), J7.6 (Pin_6)
- new net ~{C_SEL4}: J5.32 (Pin_32), J7.5 (Pin_5)
- new net ~{C_STEP}: J5.24 (Pin_24), U6.2
- new net ~{C_TRACK00}: J5.10 (Pin_10), RN2.3 (R2), U4.3 (A2)
- new net ~{C_WRFAULT}: J5.12 (Pin_12), RN2.4 (R3), U4.4 (A3)
- new net ~{C_WRITE}: J5.6 (Pin_6), U5.6
Other:
- moved on the sheet: A1, C1, J1, J4, P1, P2, RN1, U1, U2A, U2B, U2C, U2D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

Commit message: Corrected SD SPI Interface . Preparations for 2nd HD
Parts:
- added C5, C6, C7, C8: 100n, symbol Device:C
- added J8: IDC_CONN20, symbol Connector_Generic:Conn_02x10_Odd_Even
- added J9: HEAD3_SEL2, symbol Connector_Generic:Conn_02x05_Counter_Clockwise
- added R5: 100, symbol Device:R
- added R6: 4k7, symbol Device:R
- added U7: ADM1491EBR, Package_SO:SOIC-14_3.9x8.7mm_P1.27mm, symbol Interface_UART:SN65HVD33DR
- U5, U6: value 74LS05 -> 74ACT05
Connections:
- net +3V3: now also A1.36 (3V3), U2.14 (VCC), U5.14 (VCC), U6.14 (VCC), C5.1, C6.1, C7.1, C8.1, R6.1, U7.13 (VCC), U7.14 (VCC)
- net CS: now also A1.22 (GPIO17); no longer A1.27 (GPIO21)
- net GNDD: now also U2.7 (GND), U5.7 (GND), U6.7 (GND), C5.2, C6.2, C7.2, C8.2, J8.11 (Pin_11), J8.12 (Pin_12), J8.15 (Pin_15), J8.16 (Pin_16), J8.19 (Pin_19), J8.2 (Pin_2), J8.20 (Pin_20), J8.4 (Pin_4), J8.6 (Pin_6), J8.8 (Pin_8), U7.6 (GND), U7.7 (GND)
- net INDEX: now also A1.27 (GPIO21); no longer A1.22 (GPIO17)
- net MISO: now also A1.25 (GPIO19); no longer A1.26 (GPIO20)
- net MOSI: now also A1.21 (GPIO16); no longer A1.25 (GPIO19)
- net WRFAULT: now also A1.26 (GPIO20); no longer A1.21 (GPIO16)
- net ~{E_HEAD3}: now also J9.5 (Pin_5); no longer RN1.2 (R1), U1.18 (B1)
- net ~{E_SEL1}: now also J9.1 (Pin_1)
- net ~{E_SEL2}: now also J9.2 (Pin_2)
- net ~{E_SEL3}: now also J9.3 (Pin_3)
- net ~{E_SEL4}: now also J9.4 (Pin_4)
- new net: J9.10 (Pin_10), J9.6 (Pin_6), J9.7 (Pin_7), J9.8 (Pin_8), J9.9 (Pin_9), RN1.2 (R1), U1.18 (B1)
- new net: R6.2, U7.3 (~{RE}), U7.4 (DE)
- new net: U7.2 (RO), U7.5 (DI)
- new net E2_READ+: J8.17 (Pin_17), U7.9 (Y)
- new net E2_READ-: J8.18 (Pin_18), U7.10 (Z)
- new net E2_WRITE+: J8.13 (Pin_13), R5.1, U7.12 (A)
- new net E2_WRITE-: J8.14 (Pin_14), R5.2, U7.11 (B)
- new net ~{E2_DRV_SEL}: J8.1 (Pin_1)
Other:
- moved on the sheet: U2G, U5G, U6G

Commit message: Power supply added. Continue on second data port
Parts:
- added D1: 1N4148, Diode_THT:D_DO-35_SOD27_P7.62mm_Horizontal, symbol Diode:1N4148
- added J10: PWR_MOLEX, symbol Connector_Generic:Conn_01x04
Connections:
- net GNDD: now also J10.2 (Pin_2), J10.3 (Pin_3)
- net MFM_DATA: now also U7.2 (RO), U7.5 (DI)
- net ~{MFM1_IN}: now reaches R6.2, U7.3 (~{RE}), U7.4 (DE)
- net at A1.39 (VSYS): now also D1.1 (K)
- new net: D1.2 (A), J10.4 (Pin_4)
- new net +12V: J10.1 (Pin_1)
